Commit message: Improve A3 sensor bridge throughput and skeleton data

File: agibot/A3/resource/a3_ultra.urdf (robot description, URDF)
Before this commit: robot a3_ultra, 37 links, 36 joints
Links:
- added link left_hand_channel_0
- added link left_hand_channel_1
- added link left_hand_channel_2
- added link left_hand_channel_3
- added link left_hand_channel_4
- added link right_hand_channel_0
- added link right_hand_channel_1
- added link right_hand_channel_2
- added link right_hand_channel_3
- added link right_hand_channel_4
Joints:
- added joint left_hand_joint_0: type fixed, parent left_hand_link, child left_hand_channel_0
- added joint left_hand_joint_1: type fixed, parent left_hand_link, child left_hand_channel_1
- added joint left_hand_joint_2: type fixed, parent left_hand_link, child left_hand_channel_2
- added joint left_hand_joint_3: type fixed, parent left_hand_link, child left_hand_channel_3
- added joint left_hand_joint_4: type fixed, parent left_hand_link, child left_hand_channel_4
- added joint right_hand_joint_0: type fixed, parent right_hand_link, child right_hand_channel_0
- added joint right_hand_joint_1: type fixed, parent right_hand_link, child right_hand_channel_1
- added joint right_hand_joint_2: type fixed, parent right_hand_link, child right_hand_channel_2
- added joint right_hand_joint_3: type fixed, parent right_hand_link, child right_hand_channel_3
- added joint right_hand_joint_4: type fixed, parent right_hand_link, child right_hand_channel_4
